Commit message: update urdf model

File: urdf/oyku_model.xacro (robot description, xacro)
@@ -29,5 +29,5 @@
       <origin xyz="0 0 0.055" rpy="0 0 0"/>
       <geometry>
-        <box size="0.155 0.2 0.075"/>
+        <box size="0.2 0.155 0.075"/>
       </geometry>
       <material name="black"/>
@@ -36,5 +36,5 @@
       <origin xyz="0 0 0" rpy="0 0 0"/>
       <geometry>
-        <box size="0.155 0.2 0.075"/>
+        <box size="0.2 0.155 0.075"/>
       </geometry>
     </collision>
@@ -106,5 +106,5 @@
     <parent link="base_link"/>
     <child link="lidar"/>
-    <origin xyz="0 0.05 0.1375" rpy="0 0 1.5708"/>
+    <origin xyz="0 0.05 0.1375" rpy="0 0 -1.5708"/>
   </joint>
 </robot>

Commit message: fix x not pointing forward in urdf model

File: urdf/oyku_model.xacro (robot description, xacro)
@@ -73,12 +73,12 @@
       <parent link="base_link"/>
       <child link="${wheel_name}"/>
-      <origin xyz="${x} ${y} 0" rpy="0 1.57 0"/>
+      <origin xyz="${x} ${y} 0" rpy="0 1.57 1.57"/>
       <axis xyz="0 0 1"/>
     </joint>
   </xacro:macro>
-  <xacro:oyku_wheel wheel_name="wheel_fl" x="${-lx}" y="${ly}" />
-  <xacro:oyku_wheel wheel_name="wheel_fr" x="${lx}" y="${ly}" />
-  <xacro:oyku_wheel wheel_name="wheel_rl" x="${-lx}" y="${-ly}" />
-  <xacro:oyku_wheel wheel_name="wheel_rr" x="${lx}" y="${-ly}" />
+  <xacro:oyku_wheel wheel_name="wheel_fl" x="${ly}" y="${lx}" />
+  <xacro:oyku_wheel wheel_name="wheel_fr" x="${ly}" y="${-lx}" />
+  <xacro:oyku_wheel wheel_name="wheel_rl" x="${-ly}" y="${lx}" />
+  <xacro:oyku_wheel wheel_name="wheel_rr" x="${-ly}" y="${-lx}" />
   <link name="lidar">
     <visual>
@@ -106,5 +106,5 @@
     <parent link="base_link"/>
     <child link="lidar"/>
-    <origin xyz="0 0.05 0.1375" rpy="0 0 -1.5708"/>
+    <origin xyz="0.05 0 0.1375" rpy="0 0 0"/>
   </joint>
 </robot>
